File: arisu.kicad_pcb (KiCad board)
At the start: 2 copper layers, 339.1 x 118.7 mm, 176 parts, among them J1 USB_B_Micro, SW1 SW_Push, SW10 SW_Push, SW11 SW_Push, SW12 SW_Push, SW13 SW_Push, SW14 SW_Push, SW15 SW_Push, SW16 SW_Push, SW17 SW_Push, SW18 SW_Push, SW19 SW_Push, SW2 SW_Push, SW20 SW_Push, SW21 SW_Push, SW22 SW_Push, SW23 SW_Push, SW24 SW_Push, SW25 SW_Push, SW26 SW_Push, SW27 SW_Push, SW28 SW_Push, SW29 SW_Push, SW3 SW_Push, SW30 SW_Push, SW31 SW_Push, SW32 SW_Push, SW33 SW_Push, SW34 SW_Push, SW35 SW_Push, SW36 SW_Push, SW37 SW_Push, SW38 SW_Push, SW39 SW_Push, SW4 SW_Push, SW40 SW_Push, SW41 SW_Push, SW42 SW_Push, SW43 SW_Push, SW44 SW_Push, SW45 SW_Push, SW46 SW_Push, SW47 SW_Push, SW48 SW_Push, SW49 SW_Push, SW5 SW_Push, SW50 SW_Push, SW51 SW_Push, SW52 SW_Push, SW53 SW_Push, SW54 SW_Push, SW55 SW_Push, SW56 SW_Push, SW57 SW_Push, SW58 SW_Push, SW59 SW_Push, SW6 SW_Push, SW60 SW_Push, SW61 SW_Push, SW62 SW_Push, SW63 SW_Push, SW64 SW_Push, SW65 SW_Push, SW66 SW_Push, SW67 SW_Push, SW7 SW_Push, SW8 SW_Push, SW9 SW_Push, U1 USBLC6-2SC6, U2 ATmega32U4-AU, Y1 Crystal_GND24

Commit message: Replace components, place RGB leds, update traces - WIP
Parts:
- removed G*** (x2): LOGO, arisu:arisu-logo
- removed GND: GND, Pin_Headers:Pin_Header_Straight_1x01_Pitch2.54mm
- removed MISO: MISO, Pin_Headers:Pin_Header_Straight_1x01_Pitch2.54mm
- removed MOSI: MOSI, Pin_Headers:Pin_Header_Straight_1x01_Pitch2.54mm
- removed PF7: PF7, Pin_Headers:Pin_Header_Straight_1x01_Pitch2.54mm
- removed RES: RES, Pin_Headers:Pin_Header_Straight_1x01_Pitch2.54mm
- removed SCK: SCK, Pin_Headers:Pin_Header_Straight_1x01_Pitch2.54mm
- removed U1: USBLC6-2SC6, TO_SOT_Packages_SMD:SOT-23-6_Handsoldering
- removed VCC: VCC, Pin_Headers:Pin_Header_Straight_1x01_Pitch2.54mm
- removed Y1: Crystal_GND24, Crystals:Crystal_SMD_SeikoEpson_FA238-4pin_3.2x2.5mm_HandSoldering
- added J2: 1x6 2.54mm, Connector_PinHeader_2.54mm:PinHeader_1x06_P2.54mm_Vertical, F.Cu at (208.3, 26.7)
- added RD1: WS2812B, LED_SMD:LED_WS2812B_PLCC4_5.0x5.0mm_P3.2mm, B.Cu at (166.7, 43.6)
- added RD10: WS2812B, LED_SMD:LED_WS2812B_PLCC4_5.0x5.0mm_P3.2mm, B.Cu at (334.8, 43.6)
- added RD11: WS2812B, LED_SMD:LED_WS2812B_PLCC4_5.0x5.0mm_P3.2mm, B.Cu at (281.1, 43.8)
- added RD12: WS2812B, LED_SMD:LED_WS2812B_PLCC4_5.0x5.0mm_P3.2mm, B.Cu at (221.9, 39.6)
- added RD2: WS2812B, LED_SMD:LED_WS2812B_PLCC4_5.0x5.0mm_P3.2mm, B.Cu at (110.0, 46.4)
- added RD3: WS2812B, LED_SMD:LED_WS2812B_PLCC4_5.0x5.0mm_P3.2mm, B.Cu at (53.1, 43.2)
- added RD4: WS2812B, LED_SMD:LED_WS2812B_PLCC4_5.0x5.0mm_P3.2mm, B.Cu at (53.4, 109.8)
- added RD5: WS2812B, LED_SMD:LED_WS2812B_PLCC4_5.0x5.0mm_P3.2mm, B.Cu at (110.0, 110.2)
- added RD6: WS2812B, LED_SMD:LED_WS2812B_PLCC4_5.0x5.0mm_P3.2mm, B.Cu at (166.6, 110.2)
- added RD7: WS2812B, LED_SMD:LED_WS2812B_PLCC4_5.0x5.0mm_P3.2mm, B.Cu at (223.2, 110.2)
- added RD8: WS2812B, LED_SMD:LED_WS2812B_PLCC4_5.0x5.0mm_P3.2mm, B.Cu at (279.8, 110.2)
- added RD9: WS2812B, LED_SMD:LED_WS2812B_PLCC4_5.0x5.0mm_P3.2mm, B.Cu at (336.4, 110.2)
- added X1: 16Mhz, Crystal:Crystal_HC49-U_Vertical, B.Cu at (195.6, 41.9)
- D1, D10, D11, D12, D13, D14, D15, D16, D17, D18, D19, D2, D20, D21, D22, D23, D24, D25, D26, D27, D28, D29, D3, D30, D31, D32, D33, D34, D35, D36, D37, D38, D39, D4, D40, D41, D42, D43, D44, D45, D46, D47, D48, D49, D5, D50, D51, D52, D53, D54, D55, D56, D57, D58, D59, D6, D60, D61, D62, D63, D64, D65, D66, D67, D7, D8, D9: footprint Diodes_SMD:D_SOD-123 -> Diode_THT:D_DO-35_SOD27_P7.62mm_Horizontal
- J1: value USB_B_Micro -> USB_B_Mini; footprint Connectors_USB:USB_Micro-B_Molex-105017-0001 -> arisu-rgb-pcb:Mini-USB-B_OMRON_XM7D-0512
- J10: renamed from PF6; footprint Pin_Headers:Pin_Header_Straight_1x01_Pitch2.54mm -> Connector_PinHeader_2.54mm:PinHeader_1x01_P2.54mm_Vertical
- J12: renamed from VCC; footprint Pin_Headers:Pin_Header_Straight_1x01_Pitch2.54mm -> Connector_PinHeader_2.54mm:PinHeader_1x01_P2.54mm_Vertical
- J13: renamed from D+; footprint Pin_Headers:Pin_Header_Straight_1x01_Pitch2.54mm -> Connector_PinHeader_2.54mm:PinHeader_1x01_P2.54mm_Vertical
- J14: renamed from D-; footprint Pin_Headers:Pin_Header_Straight_1x01_Pitch2.54mm -> Connector_PinHeader_2.54mm:PinHeader_1x01_P2.54mm_Vertical
- J15: renamed from GND; footprint Pin_Headers:Pin_Header_Straight_1x01_Pitch2.54mm -> Connector_PinHeader_2.54mm:PinHeader_1x01_P2.54mm_Vertical
- J8: renamed from PF4; footprint Pin_Headers:Pin_Header_Straight_1x01_Pitch2.54mm -> Connector_PinHeader_2.54mm:PinHeader_1x01_P2.54mm_Vertical
- J9: renamed from PF5; footprint Pin_Headers:Pin_Header_Straight_1x01_Pitch2.54mm -> Connector_PinHeader_2.54mm:PinHeader_1x01_P2.54mm_Vertical
- SWR1: footprint Buttons_Switches_SMD:SW_SPST_TL3342 -> Button_Switch_SMD:SW_SPST_TL3342
- U2: footprint Housings_QFP:TQFP-44_10x10mm_Pitch0.8mm -> Package_QFP:TQFP-44_10x10mm_P0.8mm
- moved D46 13.4 mm to (263.0, 121.0)
- moved D2 6.54 mm to (38.2, 62.5)
- moved D7 6.03 mm to (62.5, 61.2)
- moved D4 5.90 mm to (37.8, 100.2)
- moved D33 5.56 mm to (182.8, 61.0)
- moved D1 5.42 mm to (38.8, 43.2)
- moved D14 5.41 mm to (89.8, 120.0)
- moved J1 5.40 mm to (175.3, 31.8), turned to 180 degrees
- moved D5 5.40 mm to (31.2, 120.0)
- moved D13 5.37 mm to (89.0, 101.5)
- moved D20 5.34 mm to (120.2, 69.2)
- moved D3 5.32 mm to (37.8, 81.2)
- moved D11 5.32 mm to (83.2, 59.5)
- moved D10 5.31 mm to (77.0, 42.0)
- moved D37 5.30 mm to (204.8, 130.7)
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Connections:
- U2 pad 32: /col3 -> RGBIN
- U2 pad 36: /PF7 -> /col3
Routing:
- net VCC: track 205.4 -> 351.0 mm, vias 9 -> 12
- net Net-(RD3-Pad2): track 0.00 -> 90.0 mm
- net Net-(RD5-Pad2): track 0.00 -> 60.0 mm, vias 0 -> 2
- net Net-(RD6-Pad2): track 0.00 -> 53.6 mm
- net Net-(RD7-Pad2): track 0.00 -> 53.0 mm, vias 0 -> 2
- net Net-(RD8-Pad2): track 0.00 -> 53.0 mm
- net Net-(RD4-Pad2): track 0.00 -> 52.9 mm
- net /PF7: track 46.3 -> 0.00 mm, vias 1 -> 0
- net GND: track 71.6 -> 42.5 mm, vias 12 -> 8
- net /row1: track 384.1 -> 398.8 mm, vias 4 -> 3
- net Net-(J1-Pad2): track 45.1 -> 31.2 mm
- net /row3: track 432.5 -> 443.4 mm
- net Net-(D46-Pad2): track 5.08 -> 15.8 mm
- net Net-(J1-Pad3): track 47.8 -> 40.9 mm, vias 0 -> 2
- net /row2: track 399.4 -> 406.0 mm, vias 4 -> 2
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